Commit message: update algorithm

File: urdf/pupbot.xacro (robot description, xacro)
@@ -1,4 +1,4 @@
 <?xml version="1.0"?>
-<robot name="quadruped_robot" xmlns:xacro="http://ros.org/wiki/xacro">
+<robot name="pupbot" xmlns:xacro="http://ros.org/wiki/xacro">
   <material name="gray">
     <color rgba="0.5 0.5 0.5 2.5"/>
@@ -21,5 +21,5 @@
       <origin xyz="0 0 0.13" rpy="0 0 0" />
       <geometry>
-        <mesh filename="package://quadruped_robot/stl/body.stl" />
+        <mesh filename="package://pupbot/stl/body.stl" />
       </geometry>
       <material name="gray" />
@@ -65,5 +65,5 @@
       <origin xyz="${xyz2}" rpy="0 0 0" />
       <geometry>
-        <mesh filename="package://quadruped_robot/stl/leg_shoulder.stl" />
+        <mesh filename="package://pupbot/stl/leg_shoulder.stl" />
       </geometry>
       <material name="gray"/>
@@ -86,9 +86,9 @@
   <!-- left leg upper -->
   <joint name="${prefix}_upper_joint" type="revolute">
-    <origin xyz="${xyz3}" rpy="${radians(-90)} ${radians(135)} 0"/>
+    <origin xyz="${xyz3}" rpy="${radians(-90)} ${radians(90)} 0"/>
     <parent link="${prefix}_shoulder_link"/>
     <child  link="${prefix}_upper_link"/>
     <axis xyz="0 0 1"/>
-    <limit lower="-1.7" upper="0.8" effort="${effort}" velocity="${velocity}"/>
+    <limit lower="-1.0" upper="2.0" effort="${effort}" velocity="${velocity}"/>
   </joint>
   <transmission name="${prefix}_upper_trans">
@@ -111,5 +111,5 @@
       <origin xyz="0 0 0" rpy="0 0 ${radians(180)}" />
       <geometry>
-        <mesh filename="package://quadruped_robot/stl/leg_upper.stl" />
+        <mesh filename="package://pupbot/stl/leg_upper.stl" />
       </geometry>
       <material name="gray"/>
@@ -132,9 +132,9 @@
   <!-- left leg lower -->
   <joint name="${prefix}_lower_joint" type="revolute">
-    <origin xyz="0 0.083 0" rpy="0 0 ${radians(-90)}"/>
+    <origin xyz="0 0.083 0" rpy="0 ${radians(180)} 0"/>
     <parent link="${prefix}_upper_link"/>
     <child  link="${prefix}_lower_link"/>
     <axis xyz="0 0 1"/>
-    <limit lower="-1.6" upper="1.5" effort="${effort}" velocity="${velocity}"/>
+    <limit lower="0.0" upper="3.0" effort="${effort}" velocity="${velocity}"/>
   </joint>
   <transmission name="${prefix}_lower_trans">
@@ -150,17 +150,17 @@
   <link name="${prefix}_lower_link">
     <inertial>
-      <origin xyz="0 0.0365 0.021" rpy="0 0 0" />
+      <origin xyz="0 0.0365 -0.021" rpy="0 ${radians(-180)} 0" />
       <mass value="0.0181437"/>
       <inertia ixx="0.00000820851" ixy="0.0" ixz="0.0" iyy="0.000000302395" iyz="0.0" izz="0.00000820851"/>
     </inertial>
     <visual>
-      <origin xyz="0 0 0.042" rpy="0 ${radians(90)} 0" />
-      <geometry>
-        <mesh filename="package://quadruped_robot/stl/leg_lower.stl" />
-      </geometry>
-      <material name="gray"/>
-    </visual>
-    <collision>
-      <origin xyz="0 0.0365 0.021" rpy="0 0 0" />
+      <origin xyz="0 0 -0.042" rpy="0 ${radians(-90)} 0" />
+      <geometry>
+        <mesh filename="package://pupbot/stl/leg_lower.stl" />
+      </geometry>
+      <material name="gray"/>
+    </visual>
+    <collision>
+      <origin xyz="0 0.0365 -0.021" rpy="0 0 0" />
       <geometry>
         <box size="0.01 0.073 0.01" />
@@ -183,5 +183,5 @@
   <link name="${prefix}_lower_ball">
     <collision>
-      <origin xyz="0 0.005 0.021" rpy="0 0 0" />
+      <origin xyz="0 0.005 -0.021" rpy="0 0 0" />
       <geometry>
         <sphere radius="0.005"/>
@@ -230,5 +230,5 @@
       <origin xyz="${xyz2}" rpy="0 0 ${radians(180)}" />
       <geometry>
-        <mesh filename="package://quadruped_robot/stl/leg_shoulder.stl" />
+        <mesh filename="package://pupbot/stl/leg_shoulder.stl" />
       </geometry>
       <material name="gray"/>
@@ -251,9 +251,9 @@
   <!-- right leg upper -->
   <joint name="${prefix}_upper_joint" type="revolute">
-    <origin xyz="${xyz3}" rpy="${radians(-90)} ${radians(135)} 0"/>
+    <origin xyz="${xyz3}" rpy="${radians(90)} ${radians(-90)} 0"/>
     <parent link="${prefix}_shoulder_link"/>
     <child  link="${prefix}_upper_link"/>
     <axis xyz="0 0 1"/>
-    <limit lower="-1.7" upper="0.8" effort="${effort}" velocity="${velocity}"/>
+    <limit lower="-2.0" upper="1.0" effort="${effort}" velocity="${velocity}"/>
   </joint>
   <transmission name="${prefix}_upper_trans">
@@ -269,17 +269,17 @@
   <link name="${prefix}_upper_link">
     <inertial>
-      <origin xyz="0 0.04 -0.015" rpy="0 0 0" />
+      <origin xyz="0 0.04 0.015" rpy="0 ${radians(180)} 0" />
       <mass value="0.1273437"/>
       <inertia ixx="0.00009550777" ixy="0.0" ixz="0.0" iyy="0.00001379556" iyz="0.0" izz="0.00009020178"/>
     </inertial>
     <visual>
-      <origin xyz="0 0 0" rpy="0 ${radians(180)} ${radians(180)}" />
-      <geometry>
-        <mesh filename="package://quadruped_robot/stl/leg_upper.stl" />
-      </geometry>
-      <material name="gray"/>
-    </visual>
-    <collision>
-      <origin xyz="0 0.04 -0.015" rpy="0 0 0" />
+      <origin xyz="0 0 0" rpy="0 ${radians(0)} ${radians(180)}" />
+      <geometry>
+        <mesh filename="package://pupbot/stl/leg_upper.stl" />
+      </geometry>
+      <material name="gray"/>
+    </visual>
+    <collision>
+      <origin xyz="0 0.04 0.015" rpy="0 0 0" />
       <geometry>
         <box size="0.02 0.09 0.03" />
@@ -297,9 +297,9 @@
   <!-- right leg lower -->
   <joint name="${prefix}_lower_joint" type="revolute">
-    <origin xyz="0 0.083 0" rpy="0 0 ${radians(-90)}"/>
+    <origin xyz="0 0.083 0" rpy="0 ${radians(180)} 0"/>
     <parent link="${prefix}_upper_link"/>
     <child  link="${prefix}_lower_link"/>
     <axis xyz="0 0 1"/>
-    <limit lower="-1.6" upper="1.5" effort="${effort}" velocity="${velocity}"/>
+    <limit lower="-3.0" upper="0.0" effort="${effort}" velocity="${velocity}"/>
   </joint>
   <transmission name="${prefix}_lower_trans">
@@ -322,5 +322,5 @@
       <origin xyz="0 0 0" rpy="0 ${radians(90)} 0" />
       <geometry>
-        <mesh filename="package://quadruped_robot/stl/leg_lower.stl" />
+        <mesh filename="package://pupbot/stl/leg_lower.stl" />
       </geometry>
       <material name="gray"/>

Commit message: add crawl gait algorithm

File: urdf/pupbot.xacro (robot description, xacro)
@@ -5,12 +5,12 @@
   </material>
   <!-- base -->
-  <link name="base_link"/>
+  <link name="world"/>
   <!-- body -->
   <joint name="base_joint" type="fixed">
-    <parent link="base_link"/>
-    <child  link="body_link"/>
+    <parent link="world"/>    <!-- <parent link="base_link"/> -->
+    <child  link="base_link"/>    <!-- <child link="body_link"/> -->
     <origin xyz="0 0 0" rpy="0 0 0"/>
   </joint>
-  <link name="body_link">
+  <link name="base_link">
     <inertial>
       <origin xyz="0 0 0.13" rpy="0 0 0"/>
@@ -32,5 +32,5 @@
     </collision>
   </link>
-  <gazebo reference="body_link">
+  <gazebo reference="base_link">    <!-- <gazebo reference="body_link"> -->
     <material>Gazebo/DarkGrey</material>
     <selfCollide>true</selfCollide>
@@ -41,5 +41,5 @@
   <joint name="${prefix}_shoulder_joint" type="revolute">
     <origin xyz="${xyz1}" rpy="0 ${radians(-90)} 0"/>
-    <parent link="body_link"/>
+    <parent link="base_link"/>    <!-- <parent link="body_link"/> -->
     <child  link="${prefix}_shoulder_link"/>
     <axis xyz="0 0 1"/>
@@ -206,5 +206,5 @@
   <joint name="${prefix}_shoulder_joint" type="revolute">
     <origin xyz="${xyz1}" rpy="0 ${radians(-90)} 0"/>
-    <parent link="body_link"/>
+    <parent link="base_link"/>    <!-- <parent link="body_link"/> -->
     <child  link="${prefix}_shoulder_link"/>
     <axis xyz="0 0 1"/>

Commit message: Update algorithm

File: urdf/pupbot.xacro (robot description, xacro)
@@ -1,9 +1,9 @@
 <?xml version="1.0"?>
 <robot name="pupbot" xmlns:xacro="http://ros.org/wiki/xacro">
-  <material name="gray">
-    <color rgba="0.5 0.5 0.5 2.5"/>
+  <material name="grey">
+    <color rgba="0.5 0.5 0.5 1.0"/>
   </material>
   <!-- base -->
-  <link name="world"/>
+  <link name="world"/>    <!-- <link name="base_link"/> -->
   <!-- body -->
   <joint name="base_joint" type="fixed">
@@ -12,5 +12,5 @@
     <origin xyz="0 0 0" rpy="0 0 0"/>
   </joint>
-  <link name="base_link">
+  <link name="base_link">    <!-- <link name="body_link"/> -->
     <inertial>
       <origin xyz="0 0 0.13" rpy="0 0 0"/>
@@ -23,5 +23,5 @@
         <mesh filename="package://pupbot/stl/body.stl" />
       </geometry>
-      <material name="gray" />
+      <material name="grey" />
     </visual>
     <collision>
@@ -67,5 +67,5 @@
         <mesh filename="package://pupbot/stl/leg_shoulder.stl" />
       </geometry>
-      <material name="gray"/>
+      <material name="grey"/>
     </visual>
     <collision>
@@ -113,5 +113,5 @@
         <mesh filename="package://pupbot/stl/leg_upper.stl" />
       </geometry>
-      <material name="gray"/>
+      <material name="grey"/>
     </visual>
     <collision>
@@ -159,5 +159,5 @@
         <mesh filename="package://pupbot/stl/leg_lower.stl" />
       </geometry>
-      <material name="gray"/>
+      <material name="grey"/>
     </visual>
     <collision>
@@ -232,5 +232,5 @@
         <mesh filename="package://pupbot/stl/leg_shoulder.stl" />
       </geometry>
-      <material name="gray"/>
+      <material name="grey"/>
     </visual>
     <collision>
@@ -278,5 +278,5 @@
         <mesh filename="package://pupbot/stl/leg_upper.stl" />
       </geometry>
-      <material name="gray"/>
+      <material name="grey"/>
     </visual>
     <collision>
@@ -324,5 +324,5 @@
         <mesh filename="package://pupbot/stl/leg_lower.stl" />
       </geometry>
-      <material name="gray"/>
+      <material name="grey"/>
     </visual>
     <collision>

Commit message: Update algorithm

File: urdf/pupbot.xacro (robot description, xacro)
@@ -12,5 +12,5 @@
     <origin xyz="0 0 0" rpy="0 0 0"/>
   </joint>
-  <link name="base_link">    <!-- <link name="body_link"/> -->
+  <link name="base_link">    <!-- <link name="body_link"> -->
     <inertial>
       <origin xyz="0 0 0.13" rpy="0 0 0"/>

Commit message: URDF modification

File: urdf/pupbot.xacro (robot description, xacro)
@@ -21,5 +21,5 @@
       <origin xyz="0 0 0.13" rpy="0 0 0" />
       <geometry>
-        <mesh filename="package://pupbot/stl/body.stl" />
+        <mesh filename="package://pupbot_ver1/stl/body.stl" />
       </geometry>
       <material name="grey" />
@@ -65,5 +65,5 @@
       <origin xyz="${xyz2}" rpy="0 0 0" />
       <geometry>
-        <mesh filename="package://pupbot/stl/leg_shoulder.stl" />
+        <mesh filename="package://pupbot_ver1/stl/leg_shoulder.stl" />
       </geometry>
       <material name="grey"/>
@@ -111,5 +111,5 @@
       <origin xyz="0 0 0" rpy="0 0 ${radians(180)}" />
       <geometry>
-        <mesh filename="package://pupbot/stl/leg_upper.stl" />
+        <mesh filename="package://pupbot_ver1/stl/leg_upper.stl" />
       </geometry>
       <material name="grey"/>
@@ -157,5 +157,5 @@
       <origin xyz="0 0 -0.042" rpy="0 ${radians(-90)} 0" />
       <geometry>
-        <mesh filename="package://pupbot/stl/leg_lower.stl" />
+        <mesh filename="package://pupbot_ver1/stl/leg_lower.stl" />
       </geometry>
       <material name="grey"/>
@@ -230,5 +230,5 @@
       <origin xyz="${xyz2}" rpy="0 0 ${radians(180)}" />
       <geometry>
-        <mesh filename="package://pupbot/stl/leg_shoulder.stl" />
+        <mesh filename="package://pupbot_ver1/stl/leg_shoulder.stl" />
       </geometry>
       <material name="grey"/>
@@ -276,5 +276,5 @@
       <origin xyz="0 0 0" rpy="0 ${radians(0)} ${radians(180)}" />
       <geometry>
-        <mesh filename="package://pupbot/stl/leg_upper.stl" />
+        <mesh filename="package://pupbot_ver1/stl/leg_upper.stl" />
       </geometry>
       <material name="grey"/>
@@ -322,5 +322,5 @@
       <origin xyz="0 0 0" rpy="0 ${radians(90)} 0" />
       <geometry>
-        <mesh filename="package://pupbot/stl/leg_lower.stl" />
+        <mesh filename="package://pupbot_ver1/stl/leg_lower.stl" />
       </geometry>
       <material name="grey"/>

Commit message: Add license clause and update posture control functionality

File: urdf/pupbot.xacro (robot description, xacro)
@@ -21,5 +21,5 @@
       <origin xyz="0 0 0.13" rpy="0 0 0" />
       <geometry>
-        <mesh filename="package://pupbot_ver1/stl/body.stl" />
+        <mesh filename="package://pupbot/stl/body.stl" />
       </geometry>
       <material name="grey" />
@@ -65,5 +65,5 @@
       <origin xyz="${xyz2}" rpy="0 0 0" />
       <geometry>
-        <mesh filename="package://pupbot_ver1/stl/leg_shoulder.stl" />
+        <mesh filename="package://pupbot/stl/leg_shoulder.stl" />
       </geometry>
       <material name="grey"/>
@@ -111,5 +111,5 @@
       <origin xyz="0 0 0" rpy="0 0 ${radians(180)}" />
       <geometry>
-        <mesh filename="package://pupbot_ver1/stl/leg_upper.stl" />
+        <mesh filename="package://pupbot/stl/leg_upper.stl" />
       </geometry>
       <material name="grey"/>
@@ -157,5 +157,5 @@
       <origin xyz="0 0 -0.042" rpy="0 ${radians(-90)} 0" />
       <geometry>
-        <mesh filename="package://pupbot_ver1/stl/leg_lower.stl" />
+        <mesh filename="package://pupbot/stl/leg_lower.stl" />
       </geometry>
       <material name="grey"/>
@@ -230,5 +230,5 @@
       <origin xyz="${xyz2}" rpy="0 0 ${radians(180)}" />
       <geometry>
-        <mesh filename="package://pupbot_ver1/stl/leg_shoulder.stl" />
+        <mesh filename="package://pupbot/stl/leg_shoulder.stl" />
       </geometry>
       <material name="grey"/>
@@ -276,5 +276,5 @@
       <origin xyz="0 0 0" rpy="0 ${radians(0)} ${radians(180)}" />
       <geometry>
-        <mesh filename="package://pupbot_ver1/stl/leg_upper.stl" />
+        <mesh filename="package://pupbot/stl/leg_upper.stl" />
       </geometry>
       <material name="grey"/>
@@ -322,5 +322,5 @@
       <origin xyz="0 0 0" rpy="0 ${radians(90)} 0" />
       <geometry>
-        <mesh filename="package://pupbot_ver1/stl/leg_lower.stl" />
+        <mesh filename="package://pupbot/stl/leg_lower.stl" />
       </geometry>
       <material name="grey"/>

Commit message: add support gazebo imu

File: urdf/pupbot.xacro (robot description, xacro)
@@ -36,4 +36,33 @@
     <selfCollide>true</selfCollide>
   </gazebo>
+  <!-- IMU -->
+  <joint name="imu_joint" type="fixed">
+    <parent link="base_link"/>
+    <child  link="imu_link"/>
+    <origin xyz="0 0 0" rpy="0 0 0"/>
+  </joint>
+  <link name="imu_link">
+    <visual>
+      <origin rpy="0 0 0" xyz="0 0 0.15815"/>
+      <geometry>
+        <box size="0.01 0.01 0.01"/>
+      </geometry>
+    </visual>
+  </link>
+  <gazebo reference="imu_link">
+    <sensor type="imu" name="imu">
+      <always_on>true</always_on>
+      <plugin filename="libgazebo_ros_imu_sensor.so" name="imu_plugin">
+        <topicName>imu</topicName>
+        <bodyName>imu_link</bodyName>
+        <updateRateHZ>10.0</updateRateHZ>
+        <gaussianNoise>0.0</gaussianNoise>
+        <xyzOffset>0 0 0</xyzOffset>
+        <rpyOffset>0 0 0</rpyOffset>
+        <frameName>imu_link</frameName>
+        <initialOrientationAsReference>false</initialOrientationAsReference>
+      </plugin>
+    </sensor>
+  </gazebo>
   <!-- left_legs macro -->
   <xacro:macro name="left_legs_macro" params="prefix xyz1 xyz2 xyz3 xyz4 effort velocity">
@@ -374,7 +403,8 @@
     </plugin>
     <plugin name="joint_state_publisher" filename="libgazebo_ros_joint_state_publisher.so">
-            <robotNamespace>/</robotNamespace>
-            <jointName>leftfront_leg_shoulder_joint, leftback_leg_shoulder_joint, rightfront_leg_shoulder_joint, rightback_leg_shoulder_joint, leftfront_leg_upper_joint, leftback_leg_upper_joint, rightfront_leg_upper_joint, rightback_leg_upper_joint, leftfront_leg_lower_joint, leftback_leg_lower_joint, rightfront_leg_lower_joint, rightback_leg_lower_joint</jointName>
-        </plugin>
+      <robotNamespace>/</robotNamespace>
+      <jointName>leftfront_leg_shoulder_joint, leftback_leg_shoulder_joint, rightfront_leg_shoulder_joint, rightback_leg_shoulder_joint, leftfront_leg_upper_joint, leftback_leg_upper_joint, rightfront_leg_upper_joint, rightback_leg_upper_joint, leftfront_leg_lower_joint, leftback_leg_lower_joint, rightfront_leg_lower_joint, rightback_leg_lower_joint</jointName>
+      <updateRate>10.0</updateRate>
+    </plugin>
   </gazebo>
 </robot>
